Commit message: pkg rcr_exam_bringup creation

File: RCR_examen_description/urdf/scara_basic_position_controller.xacro (robot description, xacro)
@@ -1,11 +1,11 @@
-<?xml version="1.0" encoding="utf-8"/>
+<?xml version="1.0" encoding="utf-8"?>
 <robot name="robot_scara" xmlns:xacro="http://ros.org/wiki/xacro"/>
 	<gazebo>
-		<plugin name="joint-state_publisher_controller" filename="libgazebo_ros_joint_state_publisher.so">
-			<!--update rate Hz-->
+		<plugin name="joint_state_publisher_controller" filename="libgazebo_ros_joint_state_publisher.so">
 			<update_rate>10</update_rate>
 			<joint_name>link_1_joint</joint_name>
 			<joint_name>link_2_joint</joint_name>
 			<joint_name>link_3_joint</joint_name>
+			<joint_name>link_P_joint</joint_name>
 		</plugin>
 	</gazebo>

File: RCR_examen_description/urdf/scara_gz_propierties.xacro (robot description, xacro)
@@ -1,3 +1,3 @@
-<?xml version="1.0" encoding="utf-8"?/
+<?xml version="1.0" encoding="utf-8"?>
 <robot name="robot_scara" xmlns:xacro="http://ros.org/wiki/xacro">
 	<gazebo reference="base_link">

File: RCR_examen_description/urdf/scara_simple_controller.xacro (robot description, xacro)
@@ -1,3 +1,3 @@
-<?xml version="1.0"/>
+<?xml version="1.0"?>
 <robot name="robot_scara" xmlns:xacro="http://ros.org/wiki/xacro">
 	<xacro:property name="package_name" value="RCR_examen_description"/>

File: RCR_examen_description/urdf/scara_urdf.xacro (robot description, xacro)
@@ -1,4 +1,11 @@
 <?xml version="1.0" encoding="utf-8"?>
 <robot name="robot_scara" xmlns:xacro="http://ros.org/wiki/xacro">
+	<link name="world">
+	</link>
+	<joint name="world_joint">
+		<parent link="world" />
+		<child link="base_link" />
+		<origin xyz="0.0 0.0 0.0" rpy="0.0 0.0 0.0" />
+	</joint>
 	<link name="base_link">
 		<visual>
@@ -117,3 +124,10 @@
 		<origin xyz="0.0 0.0 0.8706" rpy="0.0 0.0 0.0" />
 	</joint>
+	<link name="P">
+	</link>
+	<joint name="link_P_joint" type="">
+		<parent link="link_3" />
+		<child link="P" />
+		<origin xyz="0.25 0.0 0.0" rpy="0.0 0.0 0.0" />
+	</joint>
 </robot>

Commit message: URDF files corrections

File: RCR_examen_description/urdf/scara_basic_position_controller.xacro (robot description, xacro)
@@ -1,6 +1,7 @@
 <?xml version="1.0" encoding="utf-8"?>
-<robot name="robot_scara" xmlns:xacro="http://ros.org/wiki/xacro"/>
+<robot name="robot_scara" xmlns:xacro="http://ros.org/wiki/xacro">
 	<gazebo>
 		<plugin name="joint_state_publisher_controller" filename="libgazebo_ros_joint_state_publisher.so">
+			<!-- Update rate Hz -->
 			<update_rate>10</update_rate>
 			<joint_name>link_1_joint</joint_name>

File: RCR_examen_description/urdf/scara_simple_controller.xacro (robot description, xacro)
@@ -1,3 +1,3 @@
-<?xml version="1.0"?>
+<?xml version="1.0" encoding="utf-8"?>
 <robot name="robot_scara" xmlns:xacro="http://ros.org/wiki/xacro">
 	<xacro:property name="package_name" value="RCR_examen_description"/>

File: RCR_examen_description/urdf/scara_urdf.xacro (robot description, xacro)
@@ -1,7 +1,6 @@
 <?xml version="1.0" encoding="utf-8"?>
 <robot name="robot_scara" xmlns:xacro="http://ros.org/wiki/xacro">
-	<link name="world">
-	</link>
-	<joint name="world_joint">
+	<link name="world"/>
+	<joint name="world_joint" type="fixed">
 		<parent link="world" />
 		<child link="base_link" />
@@ -124,7 +123,6 @@
 		<origin xyz="0.0 0.0 0.8706" rpy="0.0 0.0 0.0" />
 	</joint>
-	<link name="P">
-	</link>
-	<joint name="link_P_joint" type="">
+	<link name="P"/>
+	<joint name="link_P_joint" type="fixed" >
 		<parent link="link_3" />
 		<child link="P" />
